File: kicad/Ethernet.kicad_pcb (KiCad board)
At the start: 4 copper layers, 50 x 21.4 mm, 35 parts, among them J1 RJ45_Halo_HFJ11-x2450E-LxxRL, J2 Conn_01x08, U1 W5500, X1 25MHz

Commit message: b
Routing:
- net Net-(J1-RD-): track 4.66 -> 11.9 mm
- net /RJ45/TXN: track 8.22 -> 13.8 mm
- net /RJ45/TXP: track 13.5 -> 15.4 mm
- net Net-(J1-RD+): track 10.8 -> 12.0 mm
Other:
- board text added: "CLK"
- board text added: "G"
- board text added: "MISO"
- board text added: "MOSI"
- board text added: "V"
- board text added: "~{CS}"
- board text added: "~{INT}"
- board text added: "~{RST}"

Commit message: updates
Routing:
- net /RJ45/RXN: track 7.00 -> 9.47 mm
- net /RJ45/RXP: track 9.10 -> 9.68 mm
